File: Circuit/KiCad/LED_DRIVER.sch (KiCad schematic (older format))
At the start: 5 parts

Commit message: EeSchema settled
Parts:
- C14: renamed from C?; footprint (none) -> Capacitors_SMD:C_0805_HandSoldering
- D10: renamed from D?; value D_Schottky -> D1FS4A; footprint (none) -> Diodes_SMD:SMB_Handsoldering
- L3: renamed from L?; footprint (none) -> Choke_SMD:Choke_SMD_10.4x10.4_H4.8
- R22: renamed from R?; footprint (none) -> Resistors_SMD:R_1206_HandSoldering
- U8: renamed from U?; footprint (none) -> Housings_SOT-89:SOT89-5_Housing_Handsoldering
