File: Circuit/PCB/PowerInput.sch (KiCad schematic (older format))
At the start: 50 parts, among them CN1 DF22L-2P, P4 SWITCH, Q1 RCX080N25, U2 TL431, U3 PC817, U4 PC817, U5 BM1P061FJ, U6 HV7802, U7 HT7750A

Commit message: change lib
Parts:
- CN1: footprint user_conn:CONN_RED_2P -> conn:CONN_RED_2P
Changed lines of the file:
@@
 F 0 "CN1" H 1550 2150 60  0000 C CNN
 F 1 "DF22L-2P" H 1550 1650 60  0000 C CNN
-F 2 "user_conn:CONN_RED_2P" H 1450 1950 60  0001 C CNN
+F 2 "conn:CONN_RED_2P" H 1450 1950 60  0001 C CNN
 F 3 "" H 1450 1950 60  0000 C CNN
 	1    1500 1950

Commit message: update pcb
Parts:
- BT1: footprint Connect:bornier2 -> conn:B2B-XH-A
- D7: footprint Diodes_SMD:SMB_Handsoldering -> Diodes_SMD:SMB_Standard
- D8: footprint Diodes_SMD:SMA_Handsoldering -> Diodes_SMD:SMB_Standard
- P4: footprint Connect:bornier4 -> conn:B4B-XH-A
- R10, R11, R12, R14, R18: footprint Resistors_SMD:R_0603_HandSoldering -> Resistors_SMD:R_0603
- R13: footprint Resistors_SMD:R_2512_HandSoldering -> Resistors_SMD:R_2512
Changed lines of the file:
@@
 F 0 "R10" V 3080 1950 50  0000 C CNN
 F 1 "180k" V 3000 1950 50  0000 C CNN
-F 2 "Resistors_SMD:R_0603_HandSoldering" V 2930 1950 30  0001 C CNN
+F 2 "Resistors_SMD:R_0603" V 2930 1950 30  0001 C CNN
 F 3 "" H 3000 1950 30  0000 C CNN
 	1    3000 1950
@@
 F 0 "R11" V 3080 2450 50  0000 C CNN
 F 1 "6.2k" V 3000 2450 50  0000 C CNN
-F 2 "Resistors_SMD:R_0603_HandSoldering" V 2930 2450 30  0001 C CNN
+F 2 "Resistors_SMD:R_0603" V 2930 2450 30  0001 C CNN
 F 3 "" H 3000 2450 30  0000 C CNN
 	1    3000 2450
@@
 F 0 "R13" V 3880 1400 50  0000 C CNN
 F 1 "0.27" V 3800 1400 50  0000 C CNN
-F 2 "Resistors_SMD:R_2512_HandSoldering" V 3730 1400 30  0001 C CNN
+F 2 "Resistors_SMD:R_2512" V 3730 1400 30  0001 C CNN
 F 3 "" H 3800 1400 30  0000 C CNN
 	1    3800 1400
@@
 F 0 "R12" V 3430 1750 50  0000 C CNN
 F 1 "2.7k" V 3350 1750 50  0000 C CNN
-F 2 "Resistors_SMD:R_0603_HandSoldering" V 3280 1750 30  0001 C CNN
+F 2 "Resistors_SMD:R_0603" V 3280 1750 30  0001 C CNN
 F 3 "" H 3350 1750 30  0000 C CNN
 	1    3350 1750
@@
 F 0 "R14" V 3980 1650 50  0000 C CNN
 F 1 "27k" V 3900 1650 50  0000 C CNN
-F 2 "Resistors_SMD:R_0603_HandSoldering" V 3830 1650 30  0001 C CNN
+F 2 "Resistors_SMD:R_0603" V 3830 1650 30  0001 C CNN
 F 3 "" H 3900 1650 30  0000 C CNN
 	1    3900 1650
@@
 F 0 "R18" V 4780 2350 50  0000 C CNN
 F 1 "27k" V 4700 2350 50  0000 C CNN
-F 2 "Resistors_SMD:R_0603_HandSoldering" V 4630 2350 30  0001 C CNN
+F 2 "Resistors_SMD:R_0603" V 4630 2350 30  0001 C CNN
 F 3 "" H 4700 2350 30  0000 C CNN
 	1    4700 2350
@@
 F 0 "BT1" H 1800 7250 50  0000 L CNN
 F 1 "Battery" H 1800 7150 50  0000 L CNN
-F 2 "Connect:bornier2" V 1700 7240 60  0001 C CNN
+F 2 "conn:B2B-XH-A" V 1700 7240 60  0001 C CNN
 F 3 "" V 1700 7240 60  0000 C CNN
 	1    1700 7200
@@
 F 0 "P4" H 2550 7150 50  0000 C CNN
 F 1 "SWITCH" V 2650 6900 50  0000 C CNN
-F 2 "Connect:bornier4" H 2550 6900 60  0001 C CNN
+F 2 "conn:B4B-XH-A" H 2550 6900 60  0001 C CNN
 F 3 "" H 2550 6900 60  0000 C CNN
 	1    2550 6900
@@
 F 0 "D8" H 4800 4200 50  0000 C CNN
 F 1 "ES1D" H 4800 4000 50  0000 C CNN
-F 2 "Diodes_SMD:SMA_Handsoldering" H 4800 4100 60  0001 C CNN
+F 2 "Diodes_SMD:SMB_Standard" H 4800 4100 60  0001 C CNN
 F 3 "" H 4800 4100 60  0000 C CNN
 	1    4800 4100
@@
 F 0 "D7" H 4600 3850 50  0000 C CNN
 F 1 "D1FS4A" H 4600 3650 50  0000 C CNN
-F 2 "Diodes_SMD:SMB_Handsoldering" H 4600 3750 60  0001 C CNN
+F 2 "Diodes_SMD:SMB_Standard" H 4600 3750 60  0001 C CNN
 F 3 "" H 4600 3750 60  0000 C CNN
 	1    4600 3750
