File: Circuit/PCB/PocketSocket.kicad_pcb (KiCad board)
At the start: 2 copper layers, 150 x 100 mm, 186 parts, among them CN1 DF22L-2P, P1 CONN_02X25, P2 UART, P3 I2C, P4 SWITCH, Q1 RCX080N25, U1 CY8CKIT-059_Target, U10 CL6807, U11 CL6807, U12 CL6807, U13 CL6807, U14 CL6807, U15 CL6807, U16 CL6807, U17 CL6807, U18 CL6807, U19 CL6807, U2 TL431, U20 CL6807, U21 CL6807, U22 CL6807, U23 CL6807, U24 CL6807, U25 CL6807, U26 CL6807, U27 CL6807, U28 CL6807, U29 CL6807, U3 PC817, U30 CL6807, U31 CL6807, U4 PC817, U5 BM1P061FJ, U6 HV7802, U7 HT7750A, U8 CL6807, U9 CL6807, Y1 24.576M, Y2 32.768k

Commit message: update pcb
Parts:
- BT1: footprint Connect:bornier2 -> conn:B2B-XH-A
- C1, C2: footprint Capacitors_SMD:C_1206_HandSoldering -> Capacitors_SMD:C_1206
- C14, C15, C16, C17, C18, C19, C20, C21, C22, C23, C24, C25, C26, C27, C28, C29, C30, C31, C32, C33, C34, C35, C36, C37: footprint Capacitors_SMD:C_0805_HandSoldering -> Capacitors_SMD:C_0805
- D10, D11, D12, D13, D14, D15, D16, D17, D18, D19, D20, D21, D22, D23, D24, D25, D26, D27, D28, D29, D30, D31, D32, D33, D7: footprint Diodes_SMD:SMB_Handsoldering -> Diodes_SMD:SMB_Standard
- D8: footprint Diodes_SMD:SMA_Handsoldering -> Diodes_SMD:SMB_Standard
- P2, P3, P4: footprint Connect:bornier4 -> conn:B4B-XH-A
- Q1: moved to F.Cu
- R10, R11, R12, R14, R18: footprint Resistors_SMD:R_0603_HandSoldering -> Resistors_SMD:R_0603
- R13: footprint Resistors_SMD:R_2512_HandSoldering -> Resistors_SMD:R_2512
- R22, R23, R24, R25, R26, R27, R28, R29, R30, R31, R32, R33, R34, R35, R36, R37, R38, R39, R40, R41, R42, R43, R44, R45: footprint Resistors_SMD:R_1206_HandSoldering -> Resistors_SMD:R_1206
- U10, U11, U12, U13, U14, U15, U16, U17, U18, U19, U20, U21, U22, U23, U24, U25, U26, U27, U28, U29, U30, U31, U8, U9: footprint Housings_SOT-89:SOT89-5_Housing_Handsoldering -> Housings_SOT-89:SOT89-5_Housing
- Y2: moved to B.Cu
- moved D6 146.0 mm to (30.8, 110.6), turned to 0 degrees
- moved U7 132.7 mm to (34.6, 103.0), turned to 270 degrees
- moved C4 130.7 mm to (36.5, 115.7)
- moved BT1 129.3 mm to (36.5, 94.1), turned to 180 degrees
- moved C13 124.9 mm to (28.3, 105.5), turned to 90 degrees
- moved D5 124.6 mm to (51.1, 164.0), turned to 0 degrees
- moved C5 124.4 mm to (51.8, 115.7)
- moved C30 123.4 mm to (61.3, 105.5), turned to 180 degrees
- moved P4 116.1 mm to (49.2, 94.1), turned to 180 degrees
- moved L1 115.6 mm to (42.2, 107.5), turned to 0 degrees
- moved D4 113.9 mm to (27.0, 158.9), turned to 0 degrees
- moved C10 111.7 mm to (42.9, 100.5), turned to 180 degrees
- moved R21 109.0 mm to (71.4, 179.2), turned to 270 degrees
- moved R20 107.4 mm to (63.8, 166.5), turned to 180 degrees
- moved R17 106.6 mm to (75.2, 165.2), turned to 0 degrees
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Connections:
- P2 pad 2: /TX -> /RX
- P2 pad 3: /RX -> /TX
- U1 pad 14: Net-(U1-Pad14) -> (no net)
- U1 pad 15: /LED_DRIVER_23/PWM -> /LED_DRIVER_7/PWM
- U1 pad 18: Net-(U1-Pad18) -> (no net)
- U1 pad 19: Net-(U1-Pad19) -> (no net)
- U1 pad 2: /LED_DRIVER_16/PWM -> /LED_DRIVER_0/PWM
- U1 pad 20: Net-(U1-Pad20) -> (no net)
- U1 pad 21: /PowerInput/Vsense -> /PowerInput/Isense
- U1 pad 22: /PowerInput/Isense -> /PowerInput/Vsense
- U1 pad 24: Net-(U1-Pad24) -> (no net)
- U1 pad 27: /LED_DRIVER_15/PWM -> /LED_DRIVER_23/PWM
- U1 pad 28: Net-(U1-Pad28) -> (no net)
- U1 pad 29: Net-(U1-Pad29) -> (no net)
- U1 pad 3: /LED_DRIVER_17/PWM -> /LED_DRIVER_1/PWM
- U1 pad 30: /LED_DRIVER_14/PWM -> /LED_DRIVER_22/PWM
- U1 pad 31: /LED_DRIVER_13/PWM -> /LED_DRIVER_21/PWM
- U1 pad 32: /LED_DRIVER_12/PWM -> /LED_DRIVER_20/PWM
- U1 pad 33: /LED_DRIVER_11/PWM -> /LED_DRIVER_19/PWM
- U1 pad 34: /LED_DRIVER_10/PWM -> /LED_DRIVER_18/PWM
- U1 pad 37: /LED_DRIVER_9/PWM -> /LED_DRIVER_17/PWM
- U1 pad 38: /LED_DRIVER_8/PWM -> /LED_DRIVER_16/PWM
- U1 pad 39: /LED_DRIVER_7/PWM -> /LED_DRIVER_15/PWM
- U1 pad 4: Net-(U1-Pad4) -> (no net)
- U1 pad 40: /LED_DRIVER_6/PWM -> /LED_DRIVER_14/PWM
- U1 pad 43: Net-(U1-Pad43) -> (no net)
- U1 pad 44: Net-(U1-Pad44) -> (no net)
- U1 pad 46: /LED_DRIVER_4/PWM -> /LED_DRIVER_13/PWM
- U1 pad 47: /LED_DRIVER_3/PWM -> /LED_DRIVER_11/PWM
- U1 pad 48: /LED_DRIVER_2/PWM -> /LED_DRIVER_10/PWM
- U1 pad 49: /LED_DRIVER_1/PWM -> /LED_DRIVER_9/PWM
- U1 pad 5: /LED_DRIVER_18/PWM -> /LED_DRIVER_2/PWM
- U1 pad 50: /LED_DRIVER_0/PWM -> /LED_DRIVER_8/PWM
- U1 pad 6: /LED_DRIVER_19/PWM -> /LED_DRIVER_3/PWM
- U1 pad 7: /LED_DRIVER_20/PWM -> /LED_DRIVER_4/PWM
- U1 pad 8: /LED_DRIVER_21/PWM -> /LED_DRIVER_5/PWM
- U1 pad 9: /LED_DRIVER_22/PWM -> /LED_DRIVER_6/PWM
- U20 pad 3: /LED_DRIVER_12/PWM -> (no net)
- U5 pad 7: Net-(U5-Pad7) -> (no net)
- U6 pad 4: Net-(U6-Pad4) -> (no net)
- U6 pad 5: Net-(U6-Pad5) -> (no net)
- U6 pad 7: Net-(U6-Pad7) -> (no net)
Routing:
- net Net-(CN1-Pad2): track 0.00 -> 25.8 mm
- net Net-(CN1-Pad1): track 0.00 -> 17.5 mm
- net GND: track 0.00 -> 17.5 mm
- net Net-(C1-Pad1): track 0.00 -> 12.2 mm
- net Net-(BT1-Pad1): track 0.00 -> 11.7 mm
- net VCC: track 0.00 -> 9.20 mm
- net Net-(C2-Pad1): track 0.00 -> 8.39 mm
- net +5V: track 0.00 -> 6.10 mm
- net Net-(R2-Pad1): track 0.00 -> 5.61 mm
- net Net-(C12-Pad2): track 0.00 -> 5.61 mm
- net /LED_DRIVER_18/PWM: track 0.00 -> 5.15 mm
- net Net-(D9-Pad1): track 0.00 -> 5.11 mm
- net (no net): track 0.00 -> 4.82 mm
- net Net-(D34-Pad2): track 0.00 -> 3.81 mm
- net /PowerInput/Vsense: track 0.00 -> 3.58 mm
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Other:
- board size 150 x 100 mm -> 100 x 100 mm

Commit message: update pcb layout
Parts:
- moved D5 6.84 mm to (53.7, 157.6), turned to 180 degrees
- moved C12 4.49 mm to (53.7, 162.7), turned to 180 degrees
- moved R7 4.49 mm to (42.9, 151.9), turned to 90 degrees
- moved R21 3.70 mm to (68.3, 177.3)
- moved Q1 2.62 mm to (61.3, 169.7)
- moved R20 2.62 mm to (61.3, 167.1)
- moved U18 2.56 mm to (95.6, 143.3)
- moved C24 2.56 mm to (96.8, 140.2)
- moved C25 2.56 mm to (96.8, 127.5)
- moved U19 2.56 mm to (95.6, 130.6)
- moved R32 2.56 mm to (100.0, 143.3)
- moved L14 2.56 mm to (98.1, 128.1)
- moved D20 2.56 mm to (96.2, 137.6)
- moved D21 2.56 mm to (96.2, 124.9)
- moved L13 2.56 mm to (98.1, 140.8)
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Routing:
- net Net-(CN1-Pad2): track 25.8 -> 0.00 mm
- net Net-(CN1-Pad1): track 17.5 -> 0.00 mm
- net GND: track 17.5 -> 0.00 mm
- net Net-(C1-Pad1): track 12.2 -> 0.00 mm
- net Net-(BT1-Pad1): track 11.7 -> 0.00 mm
- net VCC: track 9.20 -> 0.00 mm
- net Net-(C2-Pad1): track 8.39 -> 0.00 mm
- net +5V: track 6.10 -> 0.00 mm
- net Net-(R2-Pad1): track 5.61 -> 0.00 mm
- net Net-(C12-Pad2): track 5.61 -> 0.00 mm
- net /LED_DRIVER_18/PWM: track 5.15 -> 0.00 mm
- net Net-(D9-Pad1): track 5.11 -> 0.00 mm
- net (no net): track 4.82 -> 0.00 mm
- net Net-(D34-Pad2): track 3.81 -> 0.00 mm
- net /PowerInput/Vsense: track 3.58 -> 0.00 mm
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
Commit message: add gerber
Parts:
- ? (x4): renamed from REF**; value MountingHole_3mm -> (none)
- C14, C15, C16, C17, C18, C19, C20, C21, C22, C23, C25, C26, C27, C28, C29, C30, C31, C32, C33, C34, C35, C36, C37: value 4.7u -> (none)
- D14, D15, D16, D17, D18, D19, D21, D22, D23, D24, D25, D26, D27, D28, D29, D30, D31, D32, D33: value D1FS4A -> (none)
- R26, R27, R28, R29, R30, R31, R33, R34, R35, R36, R37, R38, R39, R40, R41, R42, R43, R44, R45: value 0.27 -> (none)
- U12, U13, U14, U15, U16, U17, U19, U20, U21, U22, U23, U24, U25, U26, U27, U28, U29, U30, U31: value CL6807 -> (none)
- moved D20 3.81 mm to (92.4, 137.6)
- moved D21 3.81 mm to (92.4, 124.9)
- moved L13 3.81 mm to (94.3, 140.8)
- moved L14 3.81 mm to (94.3, 128.1)
- moved R32 3.81 mm to (96.2, 143.3)
- moved R33 3.81 mm to (96.2, 130.6)
- moved U18 3.81 mm to (91.8, 143.3)
- moved U19 3.81 mm to (91.8, 130.6)
- moved C24 3.81 mm to (93.0, 140.2)
- moved C25 3.81 mm to (93.0, 127.5)
Routing:
- net GND: track 0.00 -> 689.4 mm, vias 0 -> 2
- net VCC: track 0.00 -> 555.2 mm, vias 0 -> 6
- net +5V: track 0.00 -> 143.0 mm
- net /LED_DRIVER_23/PWM: track 0.00 -> 102.6 mm, vias 0 -> 1
- net Net-(P1-Pad26): track 0.00 -> 81.9 mm, vias 0 -> 1
- net /LED_DRIVER_2/PWM: track 0.00 -> 81.9 mm
- net /LED_DRIVER_4/LEDA: track 0.00 -> 81.3 mm, vias 0 -> 1
- net Net-(C9-Pad1): track 0.00 -> 77.6 mm, vias 0 -> 2
- net /LED_DRIVER_5/LEDA: track 0.00 -> 72.5 mm, vias 0 -> 1
- net /LED_DRIVER_20/LEDA: track 0.00 -> 69.0 mm, vias 0 -> 1
- net /LED_DRIVER_6/LEDA: track 0.00 -> 67.2 mm, vias 0 -> 1
- net /LED_DRIVER_4/LEDC: track 0.00 -> 66.2 mm
- net /LED_DRIVER_19/PWM: track 0.00 -> 65.1 mm, vias 0 -> 2
- net /LED_DRIVER_22/PWM: track 0.00 -> 64.9 mm, vias 0 -> 2
- net /LED_DRIVER_1/PWM: track 0.00 -> 63.9 mm
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- added copper zone on B.Cu, net GND
- added copper zone on F.Cu, net GND
Other:
- outline, holes or cut-outs redrawn
- net class 30V added: clearance 0.4, trace_width 1, via_dia 1, via_drill 0.6
- net class 5V added: clearance 0.2, trace_width 0.5, via_dia 0.5, via_drill 0.4
- net class Default: trace_width 0.25 -> 0.2; via_dia 0.6 -> 0.4; via_drill 0.4 -> 0.3
- net class LED added: clearance 0.2, trace_width 0.4, via_dia 0.4, via_drill 0.3
